Commit message: Add comment: added xacro function for modularity

File: src/my_robot_description/urdf/my_robot.urdf.xacro (robot description, xacro)
@@ -1,4 +1,5 @@
 <?xml version="1.0"?>
-<robot name="my_robot">
+<robot name="my_robot" xmlns:xacro="http://www.ros.org/wiki/xacro">
+    <!-- Added xacro function for modularity -->
     <material name="red">
         <color rgba="1 0 0 1" />
@@ -10,10 +11,30 @@
         <color rgba="0.5 0.5 0.5 1" />
     </material>
+    <!-- Xacro properties -->
+    <xacro:property name="wheel_radius" value="0.1" />
+    <xacro:property name="wheel_length" value="0.05" />
+    <xacro:property name="base_length" value="0.6" />
+    <xacro:property name="base_width" value="0.4" />
+    <xacro:property name="base_height" value="0.2" />
+    <xacro:property name="wheel_x_offset" value="${base_length/4}" />
+    <xacro:property name="wheel_y_offset" value="${base_width/2 + 0.025}" />
+    <xacro:property name="castor_x_offset" value="${base_length/3}" />
+    <xacro:macro name="wheel_visual" params="name">
+        <link name="${name}_link">
+            <visual>
+                <geometry>
+                    <cylinder radius="${wheel_radius}" length="${wheel_length}" />
+                </geometry>
+                <origin xyz="0 0 0" rpy="1.5708 0 0" />
+                <material name="grey"/>
+            </visual>
+        </link>
+    </xacro:macro>
     <link name="base_link">
         <visual>
             <geometry>
-                <box size="0.6 0.4 0.2" />
+                <box size="${base_length} ${base_width} ${base_height}" />
             </geometry>
-            <origin xyz="0 0 0.1" rpy="0 0 0" />
+            <origin xyz="0 0 ${base_height/2}" rpy="0 0 0" />
         <material name="blue"/>
         </visual>
@@ -21,22 +42,6 @@
     <link name="base_footprint_link">
     </link>
-    <link name="right_wheel_link">
-        <visual>
-            <geometry>
-                <cylinder radius="0.1" length="0.05" />
-            </geometry>
-            <origin xyz="0 0 0" rpy="1.5708 0 0" />
-            <material name="grey"/>
-        </visual>
-    </link>
-    <link name="left_wheel_link">
-        <visual>
-            <geometry>
-                <cylinder radius="0.1" length="0.05" />
-            </geometry>
-            <origin xyz="0 0 0" rpy="1.5708 0 0" />
-            <material name="grey"/>
-        </visual>
-    </link>
+    <xacro:wheel_visual name="right_wheel"/>
+    <xacro:wheel_visual name="left_wheel"/>
     <link name="castor_wheel_link">
         <visual>
@@ -51,5 +56,5 @@
         <parent link="base_link"/>
         <child link="right_wheel_link"/>
-        <origin xyz="-0.15 -0.225 0" rpy="3.14159 0 0"/>
+        <origin xyz="-${wheel_x_offset} -${wheel_y_offset} 0" rpy="0 0 0"/>
         <axis xyz="0 1 0"/>
     </joint>
@@ -57,5 +62,5 @@
         <parent link="base_link"/>
         <child link="left_wheel_link"/>
-        <origin xyz="-0.15 0.225 0" rpy="0 0 0"/>
+        <origin xyz="-${wheel_x_offset} ${wheel_y_offset} 0" rpy="0 0 0"/>
         <axis xyz="0 1 0"/>
     </joint>
@@ -63,5 +68,5 @@
         <parent link="base_link"/>
         <child link="castor_wheel_link"/>
-        <origin xyz="0.2 0 0" rpy="0 0 0"/>
+        <origin xyz="${castor_x_offset} 0 0" rpy="0 0 0"/>
     </joint>
     <joint name="base_joint" type="fixed">

Commit message: added gazebo simulaition

File: src/my_robot_description/urdf/my_robot.urdf.xacro (robot description, xacro)
@@ -2,78 +2,5 @@
 <!-- Dummy commit -->
 <robot name="my_robot" xmlns:xacro="http://www.ros.org/wiki/xacro">
-    <!-- Added xacro function for modularity -->
-    <material name="red">
-        <color rgba="1 0 0 1" />
-    </material>
-    <material name="blue">
-        <color rgba="0 0 1 1" />
-    </material>
-    <material name="grey">
-        <color rgba="0.5 0.5 0.5 1" />
-    </material>
-    <!-- Xacro properties -->
-    <xacro:property name="wheel_radius" value="0.1" />
-    <xacro:property name="wheel_length" value="0.05" />
-    <xacro:property name="base_length" value="0.6" />
-    <xacro:property name="base_width" value="0.4" />
-    <xacro:property name="base_height" value="0.2" />
-    <xacro:property name="wheel_x_offset" value="${base_length/4}" />
-    <xacro:property name="wheel_y_offset" value="${base_width/2 + 0.025}" />
-    <xacro:property name="castor_x_offset" value="${base_length/3}" />
-    <xacro:macro name="wheel_visual" params="name">
-        <link name="${name}_link">
-            <visual>
-                <geometry>
-                    <cylinder radius="${wheel_radius}" length="${wheel_length}" />
-                </geometry>
-                <origin xyz="0 0 0" rpy="1.5708 0 0" />
-                <material name="grey"/>
-            </visual>
-        </link>
-    </xacro:macro>
-    <link name="base_link">
-        <visual>
-            <geometry>
-                <box size="${base_length} ${base_width} ${base_height}" />
-            </geometry>
-            <origin xyz="0 0 ${base_height/2}" rpy="0 0 0" />
-        <material name="blue"/>
-        </visual>
-    </link>
-    <link name="base_footprint_link">
-    </link>
-    <xacro:wheel_visual name="right_wheel"/>
-    <xacro:wheel_visual name="left_wheel"/>
-    <link name="castor_wheel_link">
-        <visual>
-            <geometry>
-                <sphere radius="0.05" />
-            </geometry>
-            <origin xyz="0 0 -0.05" rpy="0 0 0" />
-            <material name="grey"/>
-        </visual>
-    </link>
-    <joint name="base_to_right_wheel" type="continuous">
-        <parent link="base_link"/>
-        <child link="right_wheel_link"/>
-        <origin xyz="-${wheel_x_offset} -${wheel_y_offset} 0" rpy="0 0 0"/>
-        <axis xyz="0 1 0"/>
-    </joint>
-    <joint name="base_to_left_wheel" type="continuous">
-        <parent link="base_link"/>
-        <child link="left_wheel_link"/>
-        <origin xyz="-${wheel_x_offset} ${wheel_y_offset} 0" rpy="0 0 0"/>
-        <axis xyz="0 1 0"/>
-    </joint>
-    <joint name="base_to_castor_wheel" type="fixed">
-        <parent link="base_link"/>
-        <child link="castor_wheel_link"/>
-        <origin xyz="${castor_x_offset} 0 0" rpy="0 0 0"/>
-    </joint>
-    <joint name="base_joint" type="fixed">
-        <parent link="base_footprint_link"/>
-        <child link="base_link"/>
-        <origin xyz="0 0 .1" rpy="0 0 0"/>
-        <axis xyz="0 0 1"/>
-    </joint>
+<xacro:include filename="common_properties.xacro"/>
+<xacro:include filename="mobile_base.xacro"/>
 </robot>
