Commit message: Update robot description, camera macro, Gazebo Sim plugin, and launch integration for ROS 2 Jazzy

File: src/my_robot_description/urdf/gazebo.xacro (robot description, xacro)
@@ -1,64 +1,33 @@
 <?xml version="1.0"?>
 <robot xmlns:xacro="http://www.ros.org/wiki/xacro">
-    <!-- Gazebo plugin for differential drive -->
-    <gazebo>
-        <plugin name="diff_drive" filename="libgazebo_ros_diff_drive.so">
-            <!-- Update rate in Hz -->
-            <update_rate>50</update_rate>
-            <!-- wheels -->
-            <left_joint>base_to_left_wheel</left_joint>
-            <right_joint>base_to_right_wheel</right_joint>
-            <!-- kinematics -->
-            <wheel_separation>0.45</wheel_separation>
-            <wheel_diameter>0.2</wheel_diameter>
-            <!-- limits -->
-            <max_wheel_torque>20</max_wheel_torque>
-            <max_wheel_acceleration>1.0</max_wheel_acceleration>
-            <!-- output -->
-            <publish_odom>true</publish_odom>
-            <publish_odom_tf>true</publish_odom_tf>
-            <odometry_frame>odom</odometry_frame>
-            <robot_base_frame>base_footprint_link</robot_base_frame>
-            <!-- Remapping -->
-            <ros>
-                <remapping>cmd_vel:=cmd_vel</remapping>
-                <remapping>odom:=odom</remapping>
-            </ros>
-            <!-- Topic to receive geometry_msgs/Twist message commands -->
-            <command_topic>cmd_vel</command_topic>
-            <!-- Topic to publish nav_msgs/Odometry messages -->
-            <odometry_topic>odom</odometry_topic>
-        </plugin>
-    </gazebo>
-    <!-- Gazebo colors and physics properties -->
-    <gazebo reference="base_link">
-        <material>Gazebo/Blue</material>
-    </gazebo>
-    <gazebo reference="right_wheel_link">
-        <material>Gazebo/Grey</material>
-        <mu1>1.0</mu1>
-        <mu2>1.0</mu2>
-        <kp>1000000.0</kp>
-        <kd>100.0</kd>
-        <minDepth>0.001</minDepth>
-        <maxVel>1.0</maxVel>
-    </gazebo>
-    <gazebo reference="left_wheel_link">
-        <material>Gazebo/Grey</material>
-        <mu1>1.0</mu1>
-        <mu2>1.0</mu2>
-        <kp>1000000.0</kp>
-        <kd>100.0</kd>
-        <minDepth>0.001</minDepth>
-        <maxVel>1.0</maxVel>
-    </gazebo>
-    <gazebo reference="castor_wheel_link">
-        <material>Gazebo/Grey</material>
-        <mu1>0.01</mu1>
-        <mu2>0.01</mu2>
-        <kp>1000000.0</kp>
-        <kd>100.0</kd>
-        <minDepth>0.001</minDepth>
-        <maxVel>1.0</maxVel>
-    </gazebo>
+  <!-- Gazebo Harmonic Diff Drive Plugin -->
+  <gazebo>
+    <plugin
+      filename="gz-sim-diff-drive-system"
+      name="gz::sim::systems::DiffDrive">
+      <!-- Joints -->
+      <left_joint>base_to_left_wheel</left_joint>
+      <right_joint>base_to_right_wheel</right_joint>
+      <!-- Kinematics -->
+      <wheel_separation>0.45</wheel_separation>
+      <wheel_radius>0.1</wheel_radius>
+      <!-- Topics -->
+      <topic>cmd_vel</topic>
+      <odom_topic>odom</odom_topic>
+      <frame_id>base_footprint_link</frame_id>
+    </plugin>
+  </gazebo>
+  <!-- Gazebo materials -->
+  <gazebo reference="base_link">
+    <material>Gazebo/Blue</material>
+  </gazebo>
+  <gazebo reference="right_wheel_link">
+    <material>Gazebo/Grey</material>
+  </gazebo>
+  <gazebo reference="left_wheel_link">
+    <material>Gazebo/Grey</material>
+  </gazebo>
+  <gazebo reference="castor_wheel_link">
+    <material>Gazebo/Grey</material>
+  </gazebo>
 </robot>
