Commit message: added ros2 controller manager

File: src/my_robot_description/urdf/common_properties.xacro (robot description, xacro)
@@ -10,4 +10,7 @@
     <material name="grey">
         <color rgba="0.5 0.5 0.5 1" />
+    </material>
+    <material name="black">
+        <color rgba="0 0 0 1" />
     </material>
     <xacro:macro name="box_inertia" params="m x y z o_xyz o_rpy">

File: src/my_robot_description/urdf/lidar.xacro (robot description, xacro)
@@ -23,5 +23,5 @@
   <!-- Lidar joint (attach to base_link) -->
   <joint name="lidar_joint" type="fixed">
-    <parent link="base_link"/>
+    <parent link="base_footprint_link"/>
     <child link="lidar_link"/>
     <origin xyz="0 0 ${base_height + lidar_height/2}" rpy="0 0 0"/>

File: src/my_robot_description/urdf/mobile_base.ros2_control.xacro (robot description, xacro)
@@ -1,20 +1,26 @@
 <?xml version="1.0"?>
-<robot xmlns:xacro="http://www.ros.org/wiki/xacro">
-  <!-- ROS 2 Control configuration for mobile base -->
-  <ros2_control name="MobileBaseHardwareInterface" type="system">
+<robot name="my_robot" xmlns:xacro="http://www.ros.org/wiki/xacro">
+  <!-- ================= ROS2 CONTROL ================= -->
+  <ros2_control name="MobileBaseHardware" type="system">
     <hardware>
-      <plugin>mock_component/GenericSystem</plugin>
-    <param name="calculate_dynamics">true</param>
+      <plugin>gz_ros2_control/GazeboSimSystem</plugin>
     </hardware>
     <joint name="base_to_left_wheel">
       <command_interface name="velocity"/>
+      <state_interface name="position"/>
       <state_interface name="velocity"/>
-      <state_interface name="position"/>
     </joint>
     <joint name="base_to_right_wheel">
       <command_interface name="velocity"/>
+      <state_interface name="position"/>
       <state_interface name="velocity"/>
-      <state_interface name="position"/>
     </joint>
   </ros2_control>
+  <!-- ================= GAZEBO PLUGIN ================= -->
+<gazebo>
+  <plugin filename="gz_ros2_control-system"
+          name="gz_ros2_control::GazeboSimROS2ControlPlugin">
+      <parameters>$(find my_robot_bringup)/config/my_robot_controllers.yaml</parameters>
+ </plugin>
+</gazebo>
 </robot>

File: src/my_robot_description/urdf/my_robot.urdf.xacro (robot description, xacro)
@@ -4,6 +4,7 @@
 <xacro:include filename="common_properties.xacro"/>
 <xacro:include filename="mobile_base.xacro"/>
+<xacro:include filename="mobile_base.ros2_control.xacro"/>
 <xacro:include filename="camera.xacro"/>
 <xacro:include filename="lidar.xacro"/>
-<xacro:include filename="mobile_base_gazebo.xacro"/>
+<!-- <xacro:include filename="mobile_base_gazebo.xacro"/> -->
 </robot>
