Commit message: Add odometry setup - robot moving with odom configuration

File: src/my_robot_description/urdf/lidar.xacro (robot description, xacro)
@@ -25,5 +25,5 @@
     <parent link="base_footprint_link"/>
     <child link="lidar_link"/>
-    <origin xyz="0 0 ${base_height + lidar_height/2}" rpy="0 0 0"/>
+    <origin xyz="0 0 ${base_height + lidar_height}" rpy="0 0 0"/>
   </joint>
   <!-- Gazebo Lidar sensor plugin -->

Commit message: Fix lidar positioning and transform tree configuration
- Fixed lidar link position to sit on top of base (z = base_height + lidar_height/2)
- Changed lidar joint parent from base_footprint_link to base_link
- Updated diff_drive_controller base_frame_id from base_link to base_footprint_link
- This ensures proper transform chain: odom → base_footprint_link → base_link → lidar

File: src/my_robot_description/urdf/lidar.xacro (robot description, xacro)
@@ -23,7 +23,7 @@
   <!-- Lidar joint (attach to base_link) -->
   <joint name="lidar_joint" type="fixed">
-    <parent link="base_footprint_link"/>
+    <parent link="base_link"/>
     <child link="lidar_link"/>
-    <origin xyz="0 0 ${base_height + lidar_height}" rpy="0 0 0"/>
+    <origin xyz="0 0 ${base_height + lidar_height/2}" rpy="0 0 0"/>
   </joint>
   <!-- Gazebo Lidar sensor plugin -->
