Commit message: added ros2 control hardware with teleop

File: src/my_robot_description/urdf/mobile_base.ros2_control.xacro (robot description, xacro)
@@ -4,5 +4,10 @@
   <ros2_control name="MobileBaseHardware" type="system">
     <hardware>
-      <plugin>gz_ros2_control/GazeboSimSystem</plugin>
+      <plugin>hardware/MyHardware</plugin>
+      <param name="serial_port">/dev/ttyUSB0</param>
+      <param name="baud_rate">115200</param>
+      <param name="counts_per_rev">1260.0</param>
+      <param name="wheel_radius">0.1</param>
+      <param name="wheel_base">0.5</param>
     </hardware>
     <joint name="base_to_left_wheel">
@@ -10,4 +15,5 @@
       <state_interface name="position"/>
       <state_interface name="velocity"/>
+      <state_interface name="effort"/>
     </joint>
     <joint name="base_to_right_wheel">
@@ -15,12 +21,19 @@
       <state_interface name="position"/>
       <state_interface name="velocity"/>
+      <state_interface name="effort"/>
     </joint>
   </ros2_control>
   <!-- ================= GAZEBO PLUGIN ================= -->
-<gazebo>
+<!-- <gazebo>
   <plugin filename="gz_ros2_control-system"
           name="gz_ros2_control::GazeboSimROS2ControlPlugin">
       <parameters>$(find my_robot_bringup)/config/my_robot_controllers.yaml</parameters>
  </plugin>
-</gazebo>
+</gazebo> -->  <!-- ================= GAZEBO PLUGIN ================= -->
+<!-- <gazebo>
+  <plugin filename="gz_ros2_control-system"
+          name="gz_ros2_control::GazeboSimROS2ControlPlugin">
+      <parameters>$(find my_robot_bringup)/config/my_robot_controllers.yaml</parameters>
+ </plugin>
+</gazebo> -->
 </robot>

File: src/my_robot_description/urdf/mobile_base.xacro (robot description, xacro)
@@ -9,4 +9,5 @@
     <xacro:property name="wheel_x_offset" value="${base_length/4}" />
     <xacro:property name="wheel_y_offset" value="${base_width/2 + 0.025}" />
+    <xacro:property name="wheel_separation" value="${wheel_y_offset * 2}" />
     <xacro:property name="castor_x_offset" value="${base_length/3}" />
     <xacro:macro name="wheel_visual" params="name">
@@ -46,5 +47,5 @@
         </collision>
     </link>
-    <link name="base_footprint_link">
+    <link name="base_footprint">
     </link>
     <xacro:wheel_visual name="right_wheel"/>
@@ -71,7 +72,6 @@
         <origin xyz="-${wheel_x_offset} -${wheel_y_offset} 0" rpy="0 0 0"/>
         <axis xyz="0 1 0"/>
-                      <!-- ADD HERE -->
-          <limit effort="10.0" velocity="10.0"/>
-  <dynamics damping="1.0" friction="1.0"/>
+        <limit effort="10.0" velocity="10.0"/>
+        <dynamics damping="1.0" friction="1.0"/>
     </joint>
     <joint name="base_to_left_wheel" type="continuous">
@@ -80,7 +80,6 @@
         <origin xyz="-${wheel_x_offset} ${wheel_y_offset} 0" rpy="0 0 0"/>
         <axis xyz="0 1 0"/>
-              <!-- ADD HERE -->
-          <limit effort="10.0" velocity="10.0"/>
-  <dynamics damping="1.0" friction="1.0"/>
+        <limit effort="10.0" velocity="10.0"/>
+        <dynamics damping="1.0" friction="1.0"/>
     </joint>
     <joint name="base_to_castor_wheel" type="fixed">
@@ -90,5 +89,5 @@
     </joint>
     <joint name="base_joint" type="fixed">
-        <parent link="base_footprint_link"/>
+        <parent link="base_footprint"/>
         <child link="base_link"/>
         <origin xyz="0 0 .1" rpy="0 0 0"/>

File: src/my_robot_description/urdf/mobile_base_gazebo.xacro (robot description, xacro)
@@ -25,5 +25,5 @@
     <odom_topic>odom</odom_topic>
     <!-- Frames -->
-    <frame_id>base_footprint_link</frame_id>
+    <frame_id>base_footprint</frame_id>
     <!-- IMPORTANT FIX -->
     <command_timeout>0.5</command_timeout>
