Commit message: Added IMU sensor for gazebo and topic

File: src/my_robot_description/urdf/imu.xacro (robot description, xacro)
@@ -23,5 +23,5 @@
     <parent link="base_link"/>
     <child link="imu_link"/>
-    <origin xyz="0 0 0.05" rpy="0 0 0"/>
+    <origin xyz="${(base_length + camera_length) / 2.0} 0 ${base_height}" rpy="0 0 0"/>
   </joint>
   <gazebo reference="imu_link">

File: src/my_robot_description/urdf/my_robot.urdf.xacro (robot description, xacro)
@@ -7,4 +7,5 @@
 <xacro:include filename="camera.xacro"/>
 <xacro:include filename="lidar.xacro"/>
+<xacro:include filename="imu.xacro"/>
 <!-- <xacro:include filename="mobile_base_gazebo.xacro"/> -->
 </robot>
