Commit message: Update launch and config files for RViz and Gazebo bridge consistency

File: src/my_robot_description/urdf/camera.xacro (robot description, xacro)
@@ -38,27 +38,27 @@
         <origin xyz="0 0 0" rpy="-1.5708 0 -1.5708"/>
     </joint>
-    <!-- Gazebo camera plugin -->
-    <gazebo reference="camera_link">
-        <material>Gazebo/Red</material>
-        <sensor name="camera" type="camera">
-            <pose>0 0 0 0 0 0</pose>
-            <visualize>true</visualize>
-            <update_rate>30</update_rate>
-            <camera>
-                <horizontal_fov>1.089</horizontal_fov>
-                <image>
-                    <format>R8G8B8</format>
-                    <width>640</width>
-                    <height>480</height>
-                </image>
-                <clip>
-                    <near>0.05</near>
-                    <far>8.0</far>
-                </clip>
-            </camera>
-            <plugin name="camera_controller" filename="libgazebo_ros_camera.so">
-                <frame_name>camera_link_optical</frame_name>
-            </plugin>
-        </sensor>
-    </gazebo>
+<gazebo reference="camera_link">
+  <material>Gazebo/Red</material>
+  <sensor name="camera" type="camera">
+    <pose>0 0 0 0 0 0</pose>
+    <visualize>true</visualize>
+    <update_rate>30</update_rate>
+    <camera>
+      <horizontal_fov>1.047</horizontal_fov>
+      <image>
+        <format>R8G8B8</format>
+        <width>640</width>
+        <height>480</height>
+      </image>
+      <clip>
+        <near>0.1</near>
+        <far>100</far>
+      </clip>
+    </camera>
+    <!-- Gazebo Harmonic Camera System -->
+    <plugin
+      filename="gz-sim-camera-system"
+      name="gz::sim::systems::Camera"/>
+  </sensor>
+</gazebo>
 </robot>

File: src/my_robot_description/urdf/mobile_base.xacro (robot description, xacro)
@@ -71,4 +71,7 @@
         <origin xyz="-${wheel_x_offset} -${wheel_y_offset} 0" rpy="0 0 0"/>
         <axis xyz="0 1 0"/>
+                      <!-- ADD HERE -->
+          <limit effort="10.0" velocity="10.0"/>
+  <dynamics damping="1.0" friction="1.0"/>
     </joint>
     <joint name="base_to_left_wheel" type="continuous">
@@ -77,4 +80,7 @@
         <origin xyz="-${wheel_x_offset} ${wheel_y_offset} 0" rpy="0 0 0"/>
         <axis xyz="0 1 0"/>
+              <!-- ADD HERE -->
+          <limit effort="10.0" velocity="10.0"/>
+  <dynamics damping="1.0" friction="1.0"/>
     </joint>
     <joint name="base_to_castor_wheel" type="fixed">

File: src/my_robot_description/urdf/my_robot.urdf.xacro (robot description, xacro)
@@ -5,4 +5,4 @@
 <xacro:include filename="mobile_base.xacro"/>
 <xacro:include filename="camera.xacro"/>
-<xacro:include filename="gazebo.xacro"/>
+<xacro:include filename="mobile_base_gazebo.xacro"/>
 </robot>

Commit message: Add lidar sensor simulation with comments to camera.xacro

File: src/my_robot_description/urdf/camera.xacro (robot description, xacro)
@@ -1,64 +1,78 @@
 <?xml version="1.0"?>
 <robot xmlns:xacro="http://www.ros.org/wiki/xacro">
-    <!-- Camera properties -->
-    <xacro:property name="camera_length" value="0.05" />
-    <xacro:property name="camera_width" value="0.05" />
-    <xacro:property name="camera_height" value="0.05" />
-    <!-- Camera link -->
-    <link name="camera_link">
-        <visual>
-            <geometry>
-                <box size="${camera_length} ${camera_width} ${camera_height}" />
-            </geometry>
-            <origin xyz="0 0 0" rpy="0 0 0" />
-            <material name="red"/>
-        </visual>
-        <collision>
-            <geometry>
-                <box size="${camera_length} ${camera_width} ${camera_height}" />
-            </geometry>
-            <origin xyz="0 0 0" rpy="0 0 0" />
-        </collision>
-        <xacro:box_inertia m="0.1" x="${camera_length}" y="${camera_width}" z="${camera_height}"
-        o_xyz="0 0 0" o_rpy="0 0 0"/>
-    </link>
-    <!-- Camera optical link -->
-    <link name="camera_link_optical">
-    </link>
-    <!-- Camera joint -->
-    <joint name="camera_joint" type="fixed">
-        <parent link="base_link"/>
-        <child link="camera_link"/>
-        <origin xyz="${base_length/2} 0 ${base_height + camera_height/2}" rpy="0 0 0"/>
-    </joint>
-    <!-- Camera optical joint -->
-    <joint name="camera_optical_joint" type="fixed">
-        <parent link="camera_link"/>
-        <child link="camera_link_optical"/>
-        <origin xyz="0 0 0" rpy="-1.5708 0 -1.5708"/>
-    </joint>
-<gazebo reference="camera_link">
-  <material>Gazebo/Red</material>
-  <sensor name="camera" type="camera">
-    <pose>0 0 0 0 0 0</pose>
-    <visualize>true</visualize>
-    <update_rate>30</update_rate>
-    <camera>
-      <horizontal_fov>1.047</horizontal_fov>
-      <image>
-        <format>R8G8B8</format>
-        <width>640</width>
-        <height>480</height>
-      </image>
-      <clip>
-        <near>0.1</near>
-        <far>100</far>
-      </clip>
-    </camera>
-    <!-- Gazebo Harmonic Camera System -->
-    <plugin
-      filename="gz-sim-camera-system"
-      name="gz::sim::systems::Camera"/>
-  </sensor>
-</gazebo>
+  <!-- ================= CAMERA PROPERTIES ================= -->
+  <xacro:property name="camera_length" value="0.05"/>
+  <xacro:property name="camera_width" value="0.05"/>
+  <xacro:property name="camera_height" value="0.05"/>
+  <!-- ================= CAMERA LINK ================= -->
+  <link name="camera_link">
+    <visual>
+      <geometry>
+        <box size="${camera_length} ${camera_width} ${camera_height}"/>
+      </geometry>
+      <material name="Grey">
+        <color rgba="0.5 0.5 0.5 1"/>
+      </material>
+    </visual>
+    <collision>
+      <geometry>
+        <box size="${camera_length} ${camera_width} ${camera_height}"/>
+      </geometry>
+    </collision>
+    <inertial>
+      <mass value="0.1"/>
+      <origin xyz="0 0 0"/>
+      <inertia
+        ixx="0.0001" ixy="0.0" ixz="0.0"
+        iyy="0.0001" iyz="0.0"
+        izz="0.0001"/>
+    </inertial>
+  </link>
+  <!-- ================= FIXED JOINT TO BASE ================= -->
+  <joint name="base_camera_joint" type="fixed">
+    <parent link="base_link"/>
+    <child link="camera_link"/>
+    <origin xyz="0.2 0 0.2" rpy="0 0 0"/>
+  </joint>
+  <!-- ================= OPTICAL FRAME ================= -->
+  <link name="camera_link_optical"/>
+  <joint name="camera_optical_joint" type="fixed">
+    <parent link="camera_link"/>
+    <child link="camera_link_optical"/>
+    <origin xyz="0 0 0" rpy="-1.5707 0 -1.5707"/>
+  </joint>
+  <!-- ================= GAZEBO SIM CAMERA SENSOR ================= -->
+  <gazebo reference="camera_link">
+    <sensor name="camera_sensor" type="camera">
+      <always_on>true</always_on>
+      <update_rate>30</update_rate>
+      <visualize>true</visualize>
+      <!-- VERY IMPORTANT FOR GZ SIM -->
+      <topic>camera</topic>
+      <camera>
+        <horizontal_fov>1.3962634</horizontal_fov>
+        <image>
+          <width>640</width>
+          <height>480</height>
+          <format>R8G8B8</format>
+        </image>
+        <clip>
+          <near>0.1</near>
+          <far>20.0</far>
+        </clip>
+        <noise>
+          <type>gaussian</type>
+          <mean>0.0</mean>
+          <stddev>0.01</stddev>
+        </noise>
+        <optical_frame>camera_link_optical</optical_frame>
+        <camera_info_topic>/camera_info</camera_info_topic>
+      </camera>
+      <always_on>true</always_on>
+      <update_rate>20</update_rate>
+      <visualize>true</visualize>
+      <topic>camera/image_raw</topic>
+      <frame_name>camera_link_optical</frame_name>
+    </sensor>
+  </gazebo>
 </robot>

Commit message: camera function added

File: src/my_robot_description/urdf/camera.xacro (robot description, xacro)
@@ -1,78 +1,59 @@
 <?xml version="1.0"?>
 <robot xmlns:xacro="http://www.ros.org/wiki/xacro">
-  <!-- ================= CAMERA PROPERTIES ================= -->
-  <xacro:property name="camera_length" value="0.05"/>
-  <xacro:property name="camera_width" value="0.05"/>
-  <xacro:property name="camera_height" value="0.05"/>
-  <!-- ================= CAMERA LINK ================= -->
-  <link name="camera_link">
-    <visual>
-      <geometry>
-        <box size="${camera_length} ${camera_width} ${camera_height}"/>
-      </geometry>
-      <material name="Grey">
-        <color rgba="0.5 0.5 0.5 1"/>
-      </material>
-    </visual>
-    <collision>
-      <geometry>
-        <box size="${camera_length} ${camera_width} ${camera_height}"/>
-      </geometry>
-    </collision>
-    <inertial>
-      <mass value="0.1"/>
-      <origin xyz="0 0 0"/>
-      <inertia
-        ixx="0.0001" ixy="0.0" ixz="0.0"
-        iyy="0.0001" iyz="0.0"
-        izz="0.0001"/>
-    </inertial>
-  </link>
-  <!-- ================= FIXED JOINT TO BASE ================= -->
-  <joint name="base_camera_joint" type="fixed">
-    <parent link="base_link"/>
-    <child link="camera_link"/>
-    <origin xyz="0.2 0 0.2" rpy="0 0 0"/>
-  </joint>
-  <!-- ================= OPTICAL FRAME ================= -->
-  <link name="camera_link_optical"/>
-  <joint name="camera_optical_joint" type="fixed">
-    <parent link="camera_link"/>
-    <child link="camera_link_optical"/>
-    <origin xyz="0 0 0" rpy="-1.5707 0 -1.5707"/>
-  </joint>
-  <!-- ================= GAZEBO SIM CAMERA SENSOR ================= -->
-  <gazebo reference="camera_link">
-    <sensor name="camera_sensor" type="camera">
-      <always_on>true</always_on>
-      <update_rate>30</update_rate>
-      <visualize>true</visualize>
-      <!-- VERY IMPORTANT FOR GZ SIM -->
-      <topic>camera</topic>
-      <camera>
-        <horizontal_fov>1.3962634</horizontal_fov>
-        <image>
-          <width>640</width>
-          <height>480</height>
-          <format>R8G8B8</format>
-        </image>
-        <clip>
-          <near>0.1</near>
-          <far>20.0</far>
-        </clip>
-        <noise>
-          <type>gaussian</type>
-          <mean>0.0</mean>
-          <stddev>0.01</stddev>
-        </noise>
-        <optical_frame>camera_link_optical</optical_frame>
-        <camera_info_topic>/camera_info</camera_info_topic>
-      </camera>
-      <always_on>true</always_on>
-      <update_rate>20</update_rate>
-      <visualize>true</visualize>
-      <topic>camera/image_raw</topic>
-      <frame_name>camera_link_optical</frame_name>
-    </sensor>
-  </gazebo>
+    <xacro:property name="camera_length" value="0.01" />
+    <xacro:property name="camera_width" value="0.1" />
+    <xacro:property name="camera_height" value="0.05" />
+    <link name="camera_link">
+        <visual>
+            <geometry>
+                <box size="${camera_length} ${camera_width} ${camera_height}" />
+            </geometry>
+            <material name="grey" />
+        </visual>
+        <collision>
+            <geometry>
+                <box size="${camera_length} ${camera_width} ${camera_height}" />
+            </geometry>
+        </collision>
+        <xacro:box_inertia m="0.1" x="${camera_length}" y="${camera_width}" z="${camera_height}"
+                           o_xyz="0 0 0" o_rpy="0 0 0" />
+    </link>
+    <joint name="base_camera_joint" type="fixed">
+        <parent link="base_link" />
+        <child link="camera_link" />
+        <origin xyz="${(base_length + camera_length) / 2.0} 0 ${base_height / 2.0}" rpy="0 0 0" />
+    </joint>
+    <link name="camera_link_optical" />
+    <joint name="camera_optical_joint" type="fixed">
+        <origin xyz="0 0 0" rpy="${-pi/2} 0 ${-pi/2}"/>
+        <parent link="camera_link"/>
+        <child link="camera_link_optical"/>
+    </joint>
+    <gazebo reference="camera_link">
+        <sensor name="camera" type="camera">
+            <camera>
+                <horizontal_fov>1.3962634</horizontal_fov>
+                <image>
+                    <width>640</width>
+                    <height>480</height>
+                    <format>R8G8B8</format>
+                </image>
+                <clip>
+                    <near>0.1</near>
+                    <far>15</far>
+                </clip>
+                <noise>
+                    <type>gaussian</type>
+                    <mean>0.0</mean>
+                    <stddev>0.007</stddev>
+                </noise>
+                <optical_frame_id>camera_link_optical</optical_frame_id>
+                <camera_info_topic>/camera_info</camera_info_topic>
+            </camera>
+            <always_on>1</always_on>
+            <update_rate>20</update_rate>
+            <visualize>true</visualize>
+            <topic>/camera</topic>
+        </sensor>
+    </gazebo>
 </robot>

File: src/my_robot_description/urdf/mobile_base_gazebo.xacro (robot description, xacro)
@@ -41,10 +41,10 @@
     <material>Gazebo/Grey</material>
   </gazebo>
-  <gazebo reference="castor_wheel_link">
+  <gazebo reference="castor_wheel_link1">
     <material>Gazebo/Grey</material>
   </gazebo>
 <gazebo>
   <plugin
-    filename="gz-joint-state-publisher-system"
+    filename="gz-sim-joint-state-publisher-system"
     name="gz::sim::systems::JointStatePublisher">
     <joint_name>base_to_left_wheel</joint_name>

File: src/my_robot_description/urdf/my_robot.urdf.xacro (robot description, xacro)
@@ -5,4 +5,5 @@
 <xacro:include filename="mobile_base.xacro"/>
 <xacro:include filename="camera.xacro"/>
+<xacro:include filename="lidar.xacro"/>
 <xacro:include filename="mobile_base_gazebo.xacro"/>
 </robot>
