Commit message: PEP code suggestion and added ekf filter launch

File: src/my_robot_description/urdf/camera.xacro (robot description, xacro)
@@ -1,35 +1,35 @@
-<?xml version="1.0"?>
-<robot xmlns:xacro="http://www.ros.org/wiki/xacro">
-    <xacro:property name="camera_length" value="0.01" />
-    <xacro:property name="camera_width" value="0.1" />
-    <xacro:property name="camera_height" value="0.05" />
-    <link name="camera_link">
+<?xml version='1.0'?>
+<robot xmlns:xacro='http://www.ros.org/wiki/xacro'>
+    <xacro:property name='camera_length' value='0.01' />
+    <xacro:property name='camera_width' value='0.1' />
+    <xacro:property name='camera_height' value='0.05' />
+    <link name='camera_link'>
         <visual>
             <geometry>
-                <box size="${camera_length} ${camera_width} ${camera_height}" />
+                <box size='${camera_length} ${camera_width} ${camera_height}' />
             </geometry>
-            <material name="grey" />
+            <material name='grey' />
         </visual>
         <collision>
             <geometry>
-                <box size="${camera_length} ${camera_width} ${camera_height}" />
+                <box size='${camera_length} ${camera_width} ${camera_height}' />
             </geometry>
         </collision>
-        <xacro:box_inertia m="0.1" x="${camera_length}" y="${camera_width}" z="${camera_height}"
-                           o_xyz="0 0 0" o_rpy="0 0 0" />
+        <xacro:box_inertia m='0.1' x='${camera_length}' y='${camera_width}' z='${camera_height}'
+                           o_xyz='0 0 0' o_rpy='0 0 0' />
     </link>
-    <joint name="base_camera_joint" type="fixed">
-        <parent link="base_link" />
-        <child link="camera_link" />
-        <origin xyz="${(base_length + camera_length) / 2.0} 0 ${base_height / 2.0}" rpy="0 0 0" />
+    <joint name='base_camera_joint' type='fixed'>
+        <parent link='base_link' />
+        <child link='camera_link' />
+        <origin xyz='${(base_length + camera_length) / 2.0} 0 ${base_height / 2.0}' rpy='0 0 0' />
     </joint>
-    <link name="camera_link_optical" />
-    <joint name="camera_optical_joint" type="fixed">
-        <origin xyz="0 0 0" rpy="${-pi/2} 0 ${-pi/2}"/>
-        <parent link="camera_link"/>
-        <child link="camera_link_optical"/>
+    <link name='camera_link_optical' />
+    <joint name='camera_optical_joint' type='fixed'>
+        <origin xyz='0 0 0' rpy='${-pi/2} 0 ${-pi/2}'/>
+        <parent link='camera_link'/>
+        <child link='camera_link_optical'/>
     </joint>
-    <gazebo reference="camera_link">
-        <sensor name="camera" type="camera">
+    <gazebo reference='camera_link'>
+        <sensor name='camera' type='camera'>
             <camera>
                 <horizontal_fov>1.3962634</horizontal_fov>

File: src/my_robot_description/urdf/imu.xacro (robot description, xacro)
@@ -1,30 +1,30 @@
-<?xml version="1.0"?>
-<robot xmlns:xacro="http://www.ros.org/wiki/xacro">
-  <link name="imu_link">
+<?xml version='1.0'?>
+<robot xmlns:xacro='http://www.ros.org/wiki/xacro'>
+  <link name='imu_link'>
     <visual>
       <geometry>
-        <box size="0.02 0.02 0.02"/>
+        <box size='0.02 0.02 0.02'/>
       </geometry>
     </visual>
     <collision>
       <geometry>
-        <box size="0.02 0.02 0.02"/>
+        <box size='0.02 0.02 0.02'/>
       </geometry>
     </collision>
     <inertial>
-      <mass value="0.01"/>
-      <origin xyz="0 0 0"/>
-      <inertia ixx="0.00001" ixy="0" ixz="0"
-               iyy="0.00001" iyz="0"
-               izz="0.00001"/>
+      <mass value='0.01'/>
+      <origin xyz='0 0 0'/>
+      <inertia ixx='0.00001' ixy='0' ixz='0'
+               iyy='0.00001' iyz='0'
+               izz='0.00001'/>
     </inertial>
   </link>
-  <joint name="imu_joint" type="fixed">
-    <parent link="base_link"/>
-    <child link="imu_link"/>
-    <origin xyz="${(base_length + camera_length) / 2.0} 0 ${base_height}" rpy="0 0 0"/>
+  <joint name='imu_joint' type='fixed'>
+    <parent link='base_link'/>
+    <child link='imu_link'/>
+    <origin xyz='${(base_length + camera_length) / 2.0} 0 ${base_height}' rpy='0 0 0'/>
   </joint>
-  <gazebo reference="imu_link">
-    <sensor name="imu_sensor" type="imu">
+  <gazebo reference='imu_link'>
+    <sensor name='imu_sensor' type='imu'>
       <always_on>true</always_on>
       <update_rate>100</update_rate>

File: src/my_robot_description/urdf/lidar.xacro (robot description, xacro)
@@ -1,33 +1,33 @@
-<?xml version="1.0"?>
-<robot xmlns:xacro="http://www.ros.org/wiki/xacro">
+<?xml version='1.0'?>
+<robot xmlns:xacro='http://www.ros.org/wiki/xacro'>
   <!-- Lidar properties -->
-  <xacro:property name="lidar_radius" value="0.05"/>
-  <xacro:property name="lidar_height" value="0.1"/>
+  <xacro:property name='lidar_radius' value='0.05'/>
+  <xacro:property name='lidar_height' value='0.1'/>
   <!-- Lidar link -->
-  <link name="lidar_link">
+  <link name='lidar_link'>
     <visual>
       <geometry>
-        <cylinder radius="${lidar_radius}" length="${lidar_height}"/>
+        <cylinder radius='${lidar_radius}' length='${lidar_height}'/>
       </geometry>
-      <origin xyz="0 0 0" rpy="0 0 0"/>
-      <material name="black"/>
+      <origin xyz='0 0 0' rpy='0 0 0'/>
+      <material name='black'/>
     </visual>
     <collision>
       <geometry>
-        <cylinder radius="${lidar_radius}" length="${lidar_height}"/>
+        <cylinder radius='${lidar_radius}' length='${lidar_height}'/>
       </geometry>
-      <origin xyz="0 0 0" rpy="0 0 0"/>
+      <origin xyz='0 0 0' rpy='0 0 0'/>
     </collision>
-    <xacro:cylinder_inertia m="0.5" r="${lidar_radius}" h="${lidar_height}" o_xyz="0 0 0" o_rpy="0 0 0"/>
+    <xacro:cylinder_inertia m='0.5' r='${lidar_radius}' h='${lidar_height}' o_xyz='0 0 0' o_rpy='0 0 0'/>
   </link>
   <!-- Lidar joint (attach to base_link) -->
-  <joint name="lidar_joint" type="fixed">
-    <parent link="base_link"/>
-    <child link="lidar_link"/>
-    <origin xyz="0 0 ${base_height + lidar_height/2}" rpy="0 0 0"/>
+  <joint name='lidar_joint' type='fixed'>
+    <parent link='base_link'/>
+    <child link='lidar_link'/>
+    <origin xyz='0 0 ${base_height + lidar_height/2}' rpy='0 0 0'/>
   </joint>
   <!-- Gazebo Lidar sensor plugin -->
-  <gazebo reference="lidar_link">
-    <sensor name="lidar" type="gpu_lidar">
+  <gazebo reference='lidar_link'>
+    <sensor name='lidar' type='gpu_lidar'>
       <gz_frame_id>lidar_link</gz_frame_id>
       <update_rate>20</update_rate>

File: src/my_robot_description/urdf/mobile_base.ros2_control.xacro (robot description, xacro)
@@ -1,36 +1,36 @@
-<?xml version="1.0"?>
-<robot name="my_robot" xmlns:xacro="http://www.ros.org/wiki/xacro">
+<?xml version='1.0'?>
+<robot name='my_robot' xmlns:xacro='http://www.ros.org/wiki/xacro'>
   <!-- ================= ROS2 CONTROL ================= -->
-  <ros2_control name="MobileBaseHardware" type="system">
+  <ros2_control name='MobileBaseHardware' type='system'>
     <hardware>
       <plugin>gz_ros2_control/GazeboSimSystem</plugin>
-      <!-- <param name="serial_port">/dev/ttyUSB0</param>
-      <param name="baud_rate">115200</param>
-      <param name="counts_per_rev">1260.0</param>
-      <param name="wheel_radius">0.035</param>
-      <param name="wheel_base">0.34</param> -->
+      <!-- <param name='serial_port'>/dev/ttyUSB0</param>
+      <param name='baud_rate'>115200</param>
+      <param name='counts_per_rev'>1260.0</param>
+      <param name='wheel_radius'>0.035</param>
+      <param name='wheel_base'>0.34</param> -->
     </hardware>
-    <joint name="base_to_left_wheel">
-      <command_interface name="velocity"/>
-      <state_interface name="position"/>
-      <state_interface name="velocity"/>
-      <state_interface name="effort"/>
+    <joint name='base_to_left_wheel'>
+      <command_interface name='velocity'/>
+      <state_interface name='position'/>
+      <state_interface name='velocity'/>
+      <state_interface name='effort'/>
     </joint>
-    <joint name="base_to_right_wheel">
-      <command_interface name="velocity"/>
-      <state_interface name="position"/>
-      <state_interface name="velocity"/>
-      <state_interface name="effort"/>
+    <joint name='base_to_right_wheel'>
+      <command_interface name='velocity'/>
+      <state_interface name='position'/>
+      <state_interface name='velocity'/>
+      <state_interface name='effort'/>
     </joint>
   </ros2_control>
   <!-- ================= GAZEBO PLUGIN ================= -->
 <!-- <gazebo>
-  <plugin filename="gz_ros2_control-system"
-          name="gz_ros2_control::GazeboSimROS2ControlPlugin">
+  <plugin filename='gz_ros2_control-system'
+          name='gz_ros2_control::GazeboSimROS2ControlPlugin'>
       <parameters>$(find my_robot_bringup)/config/my_robot_controllers.yaml</parameters>
  </plugin>
 </gazebo> -->  <!-- ================= GAZEBO PLUGIN ================= -->
 <gazebo>
-  <plugin filename="/opt/ros/jazzy/lib/libgz_ros2_control-system.so" name="gz_ros2_control::GazeboSimROS2ControlPlugin">
+  <plugin filename='/opt/ros/jazzy/lib/libgz_ros2_control-system.so' name='gz_ros2_control::GazeboSimROS2ControlPlugin'>
       <parameters>$(find my_robot_bringup)/config/my_robot_controllers.yaml</parameters>
  </plugin>

File: src/my_robot_description/urdf/mobile_base.xacro (robot description, xacro)
@@ -1,96 +1,96 @@
-<?xml version="1.0"?>
-<robot name="my_robot" xmlns:xacro="http://www.ros.org/wiki/xacro">
+<?xml version='1.0'?>
+<robot name='my_robot' xmlns:xacro='http://www.ros.org/wiki/xacro'>
     <!-- Xacro properties -->
-    <xacro:property name="wheel_radius" value="0.1" />
-    <xacro:property name="wheel_length" value="0.05" />
-    <xacro:property name="base_length" value="0.6" />
-    <xacro:property name="base_width" value="0.4" />
-    <xacro:property name="base_height" value="0.2" />
-    <xacro:property name="wheel_x_offset" value="${base_length/4}" />
-    <xacro:property name="wheel_y_offset" value="${base_width/2 + 0.025}" />
-    <xacro:property name="wheel_separation" value="${wheel_y_offset * 2}" />
-    <xacro:property name="castor_x_offset" value="${base_length/3}" />
-    <xacro:macro name="wheel_visual" params="name">
-        <link name="${name}_link">
+    <xacro:property name='wheel_radius' value='0.1' />
+    <xacro:property name='wheel_length' value='0.05' />
+    <xacro:property name='base_length' value='0.6' />
+    <xacro:property name='base_width' value='0.4' />
+    <xacro:property name='base_height' value='0.2' />
+    <xacro:property name='wheel_x_offset' value='${base_length/4}' />
+    <xacro:property name='wheel_y_offset' value='${base_width/2 + 0.025}' />
+    <xacro:property name='wheel_separation' value='${wheel_y_offset * 2}' />
+    <xacro:property name='castor_x_offset' value='${base_length/3}' />
+    <xacro:macro name='wheel_visual' params='name'>
+        <link name='${name}_link'>
             <visual>
                 <geometry>
-                    <cylinder radius="${wheel_radius}" length="${wheel_length}" />
+                    <cylinder radius='${wheel_radius}' length='${wheel_length}' />
                 </geometry>
-                <origin xyz="0 0 0" rpy="1.5708 0 0" />
-                <material name="grey"/>
+                <origin xyz='0 0 0' rpy='1.5708 0 0' />
+                <material name='grey'/>
             </visual>
-            <xacro:cylinder_inertia m="1.0" r="${wheel_radius}" h="${wheel_length}"
-            o_xyz="0 0 0" o_rpy="1.5708 0 0"/>
+            <xacro:cylinder_inertia m='1.0' r='${wheel_radius}' h='${wheel_length}'
+            o_xyz='0 0 0' o_rpy='1.5708 0 0'/>
             <collision>
                 <geometry>
-                    <cylinder radius="${wheel_radius}" length="${wheel_length}" />
+                    <cylinder radius='${wheel_radius}' length='${wheel_length}' />
                 </geometry>
-                <origin xyz="0 0 0" rpy="1.5708 0 0" />
+                <origin xyz='0 0 0' rpy='1.5708 0 0' />
             </collision>
         </link>
     </xacro:macro>
-    <link name="base_link">
+    <link name='base_link'>
         <visual>
             <geometry>
-                <box size="${base_length} ${base_width} ${base_height}" />
+                <box size='${base_length} ${base_width} ${base_height}' />
             </geometry>
-            <origin xyz="0 0 ${base_height/2}" rpy="0 0 0" />
-        <material name="blue"/>
+            <origin xyz='0 0 ${base_height/2}' rpy='0 0 0' />
+        <material name='blue'/>
         </visual>
-        <xacro:box_inertia m="5.0" x="${base_length}" y="${base_width}" z="${base_height}"
-        o_xyz="0 0 ${base_height/2}" o_rpy="0 0 0"/>
+        <xacro:box_inertia m='5.0' x='${base_length}' y='${base_width}' z='${base_height}'
+        o_xyz='0 0 ${base_height/2}' o_rpy='0 0 0'/>
         <collision>
             <geometry>
-                <box size="${base_length} ${base_width} ${base_height}" />
+                <box size='${base_length} ${base_width} ${base_height}' />
             </geometry>
-            <origin xyz="0 0 ${base_height/2}" rpy="0 0 0" />
+            <origin xyz='0 0 ${base_height/2}' rpy='0 0 0' />
         </collision>
     </link>
-    <link name="base_footprint">
+    <link name='base_footprint'>
     </link>
-    <xacro:wheel_visual name="right_wheel"/>
-    <xacro:wheel_visual name="left_wheel"/>
-    <link name="castor_wheel_link">
+    <xacro:wheel_visual name='right_wheel'/>
+    <xacro:wheel_visual name='left_wheel'/>
+    <link name='castor_wheel_link'>
         <visual>
             <geometry>
-                <sphere radius="0.05" />
+                <sphere radius='0.05' />
             </geometry>
-            <origin xyz="0 0 -0.05" rpy="0 0 0" />
-            <material name="grey"/>
+            <origin xyz='0 0 -0.05' rpy='0 0 0' />
+            <material name='grey'/>
         </visual>
-        <xacro:sphere_inertia m="0.5" r="0.05" o_xyz="0 0 -0.05" o_rpy="0 0 0"/>
+        <xacro:sphere_inertia m='0.5' r='0.05' o_xyz='0 0 -0.05' o_rpy='0 0 0'/>
         <collision>
             <geometry>
-                <sphere radius="0.05" />
+                <sphere radius='0.05' />
             </geometry>
-            <origin xyz="0 0 -0.05" rpy="0 0 0" />
+            <origin xyz='0 0 -0.05' rpy='0 0 0' />
         </collision>
     </link>
-    <joint name="base_to_right_wheel" type="continuous">
-        <parent link="base_link"/>
-        <child link="right_wheel_link"/>
-        <origin xyz="-${wheel_x_offset} -${wheel_y_offset} 0" rpy="0 0 0"/>
-        <axis xyz="0 1 0"/>
-        <limit effort="10.0" velocity="10.0"/>
-        <dynamics damping="1.0" friction="1.0"/>
+    <joint name='base_to_right_wheel' type='continuous'>
+        <parent link='base_link'/>
+        <child link='right_wheel_link'/>
+        <origin xyz='-${wheel_x_offset} -${wheel_y_offset} 0' rpy='0 0 0'/>
+        <axis xyz='0 1 0'/>
+        <limit effort='10.0' velocity='10.0'/>
+        <dynamics damping='1.0' friction='1.0'/>
     </joint>
-    <joint name="base_to_left_wheel" type="continuous">
-        <parent link="base_link"/>
-        <child link="left_wheel_link"/>
-        <origin xyz="-${wheel_x_offset} ${wheel_y_offset} 0" rpy="0 0 0"/>
-        <axis xyz="0 1 0"/>
-        <limit effort="10.0" velocity="10.0"/>
-        <dynamics damping="1.0" friction="1.0"/>
+    <joint name='base_to_left_wheel' type='continuous'>
+        <parent link='base_link'/>
+        <child link='left_wheel_link'/>
+        <origin xyz='-${wheel_x_offset} ${wheel_y_offset} 0' rpy='0 0 0'/>
+        <axis xyz='0 1 0'/>
+        <limit effort='10.0' velocity='10.0'/>
+        <dynamics damping='1.0' friction='1.0'/>
     </joint>
-    <joint name="base_to_castor_wheel" type="fixed">
-        <parent link="base_link"/>
-        <child link="castor_wheel_link"/>
-        <origin xyz="${castor_x_offset} 0 0" rpy="0 0 0"/>
+    <joint name='base_to_castor_wheel' type='fixed'>
+        <parent link='base_link'/>
+        <child link='castor_wheel_link'/>
+        <origin xyz='${castor_x_offset} 0 0' rpy='0 0 0'/>
     </joint>
-    <joint name="base_joint" type="fixed">
-        <parent link="base_footprint"/>
-        <child link="base_link"/>
-        <origin xyz="0 0 .1" rpy="0 0 0"/>
-        <axis xyz="0 0 1"/>
+    <joint name='base_joint' type='fixed'>
+        <parent link='base_footprint'/>
+        <child link='base_link'/>
+        <origin xyz='0 0 .1' rpy='0 0 0'/>
+        <axis xyz='0 0 1'/>
     </joint>
 </robot>

File: src/my_robot_description/urdf/my_robot.urdf.xacro (robot description, xacro)
@@ -1,11 +1,11 @@
-<?xml version="1.0"?>
+<?xml version='1.0'?>
 <!-- Dummy commit -->
-<robot name="my_robot" xmlns:xacro="http://www.ros.org/wiki/xacro">
-<xacro:include filename="common_properties.xacro"/>
-<xacro:include filename="mobile_base.xacro"/>
-<xacro:include filename="mobile_base.ros2_control.xacro"/>
-<xacro:include filename="camera.xacro"/>
-<xacro:include filename="lidar.xacro"/>
-<xacro:include filename="imu.xacro"/>
-<!-- <xacro:include filename="mobile_base_gazebo.xacro"/> -->
+<robot name='my_robot' xmlns:xacro='http://www.ros.org/wiki/xacro'>
+<xacro:include filename='common_properties.xacro'/>
+<xacro:include filename='mobile_base.xacro'/>
+<xacro:include filename='mobile_base.ros2_control.xacro'/>
+<xacro:include filename='camera.xacro'/>
+<xacro:include filename='lidar.xacro'/>
+<xacro:include filename='imu.xacro'/>
+<!-- <xacro:include filename='mobile_base_gazebo.xacro'/> -->
 </robot>
