Commit message: Fix package.xml dependency gaps, switch Dockerfile to rosdep-driven install, and fix odometry drift
- Audit and fix missing/unused rosdep dependencies across all packages (launch,
  launch_ros, ament_index_python, joy, joint_state_broadcaster,
  diff_drive_controller, libboost-system-dev, etc.)
- Replace hand-maintained ROS package list in docker/Dockerfile with
  `rosdep install --from-paths src --ignore-src`, using package.xml as the
  single source of truth; keep PC-only Gazebo packages and explore_lite
  (no rosdep key yet) handled separately
- Remove unused turtlebot3 packages from Dockerfile
- Fix duplicate transform_tolerance key in amcl_params.yaml that was
  silently overriding the intended value
- Fix wheel_separation_multiplier (1.41 -> 1.0) in diff_drive_controller
  config; URDF geometry already gives the correct 0.35m wheel separation,
  so the multiplier was inflating it and causing heading drift during turns
- Add new SLAM maps (industrial-warehouse, ionic) and Gazebo worlds
  (Ionic_World, living_room)
- Remove tracked .env file and ignore it, plus *.core and .claude/, going
  forward

Co-Authored-By: Claude Sonnet 4.6 <noreply@anthropic.com>

File: src/my_robot_description/urdf/camera.xacro (robot description, xacro)
@@ -52,5 +52,5 @@
             </camera>
             <always_on>1</always_on>
-            <update_rate>20</update_rate>
+            <update_rate>100</update_rate>
             <visualize>true</visualize>
             <topic>/camera</topic>

File: src/my_robot_description/urdf/lidar.xacro (robot description, xacro)
@@ -31,5 +31,5 @@
     <sensor name='lidar' type='gpu_lidar'>
       <gz_frame_id>lidar_link</gz_frame_id>
-      <update_rate>20</update_rate>
+      <update_rate>100</update_rate>
       <visualize>true</visualize>
       <visualize_type>rays</visualize_type>

File: src/my_robot_description/urdf/mobile_base.ros2_control.xacro (robot description, xacro)
@@ -4,5 +4,5 @@
   <ros2_control name='MobileBaseHardware' type='system'>
     <hardware>
-      <plugin>hardware/MyHardware</plugin>
+      <plugin>gz_ros2_control/GazeboSimSystem</plugin>
       <!-- <param name='serial_port'>/dev/ttyUSB0</param>
       <param name='baud_rate'>115200</param>

File: src/my_robot_description/urdf/mobile_base.xacro (robot description, xacro)
@@ -9,12 +9,12 @@
     <xacro:property name='wheel_x_offset' value='${base_length/4}' />
     <xacro:property name='wheel_y_offset' value='${base_width/2 + 0.025}' />
-    <xacro:property name='wheel_separation' value='.34' />
+    <xacro:property name='wheel_separation' value='.35' />
     <xacro:property name='castor_radius' value='0.05' />
     <xacro:property name='castor_length' value='0.1' />
-    <xacro:property name='castor_wheel_radius' value='0.04' />
+    <xacro:property name='castor_wheel_radius' value='0.05' />
     <xacro:property name='castor_wheel_length' value='0.02' />
     <xacro:property name='castor_x_offset' value='${base_length/3}' />
     <xacro:property name='castor_y_offset' value='0' />
-    <xacro:property name='castor_z_offset' value='0' />
+    <xacro:property name='castor_z_offset' value='${castor_wheel_radius/2 - wheel_radius}' />
     <xacro:macro name='wheel_visual' params='name'>
         <link name='${name}_link'>
@@ -25,4 +25,12 @@
                 <origin xyz='0 0 0' rpy='1.5708 0 0' />
                 <material name='grey'/>
+            </visual>
+            <!-- Stripe marker across the wheel face so rotation is visible in the viewport -->
+            <visual>
+                <geometry>
+                    <box size='${2*wheel_radius + 0.01} 0.01 ${wheel_length + 0.005}' />
+                </geometry>
+                <origin xyz='0 0 0' rpy='1.5708 0 0' />
+                <material name='red'/>
             </visual>
             <xacro:cylinder_inertia m='1.0' r='${wheel_radius}' h='${wheel_length}'
@@ -60,13 +68,13 @@
         <visual>
             <geometry>
-                <sphere radius='${castor_wheel_radius}' />
+                <sphere radius='${castor_wheel_radius/2}' />
             </geometry>
             <origin xyz='0 0 0' rpy='0 0 0' />
             <material name='grey'/>
         </visual>
-        <xacro:sphere_inertia m='0.5' r='${castor_wheel_radius}' o_xyz='0 0 -${castor_wheel_radius}' o_rpy='0 0 0'/>
+        <xacro:sphere_inertia m='0.5' r='${castor_wheel_radius/2}' o_xyz='0 0 0' o_rpy='0 0 0'/>
         <collision>
             <geometry>
-                <sphere radius='${castor_wheel_radius}' />
+                <sphere radius='${castor_wheel_radius/2}' />
             </geometry>
             <origin xyz='0 0 0' rpy='0 0 0' />
@@ -78,6 +86,6 @@
         <origin xyz='-${wheel_x_offset} -${wheel_y_offset} 0' rpy='0 0 0'/>
         <axis xyz='0 1 0'/>
-        <limit effort='10.0' velocity='10.0'/>
-        <dynamics damping='1.0' friction='1.0'/>
+        <!-- <limit effort='10.0' velocity='10.0'/> -->
+        <!-- <dynamics damping="0.01" friction="0.00"/> -->
     </joint>
     <joint name='base_to_left_wheel' type='continuous'>
@@ -86,11 +94,11 @@
         <origin xyz='-${wheel_x_offset} ${wheel_y_offset} 0' rpy='0 0 0'/>
         <axis xyz='0 1 0'/>
-        <limit effort='10.0' velocity='10.0'/>
-        <dynamics damping='1.0' friction='1.0'/>
+        <!-- <limit effort='10.0' velocity='10.0'/> -->
+        <!-- <dynamics damping='0.01' friction='0.00'/> -->
     </joint>
     <joint name='base_to_castor_wheel' type='fixed'>
         <parent link='base_link'/>
         <child link='castor_wheel_link'/>
-        <origin xyz='${castor_x_offset} ${castor_y_offset} ${castor_z_offset}' rpy='0 0 0'/>
+        <origin xyz='${castor_x_offset} ${castor_y_offset} ${castor_z_offset}' rpy='0 0 ${castor_z_offset}'/>
     </joint>
     <joint name='base_joint' type='fixed'>

File: src/my_robot_description/urdf/mobile_base_gazebo.xacro (robot description, xacro)
@@ -1,56 +1,30 @@
 <?xml version="1.0"?>
 <robot xmlns:xacro="http://www.ros.org/wiki/xacro">
-<!-- <gazebo reference="castor_wheel_link">
-    <multi_friction>
-        <friction>
-            <ode>
-                <mu>0.8</mu>
-                <mu2>0.8</mu2>
-            </ode>
-        </friction>
-    </multi_friction>
-  </gazebo> -->
-<!-- Gazebo diff-drive plugin removed to avoid duplicate control with ROS2 diff_drive_controller.
-<gazebo>
-  <plugin
-    filename="gz-sim-diff-drive-system"
-    name="gz::sim::systems::DiffDrive">
-    <!-- Joints -->
-    <left_joint>base_to_left_wheel</left_joint>
-    <right_joint>base_to_right_wheel</right_joint>
-    <!-- Robot geometry -->
-    <wheel_separation>0.35</wheel_separation>
-    <wheel_radius>0.04</wheel_radius>
-    <!-- Topics -->
-    <topic>cmd_vel</topic>
-    <odom_topic>odom</odom_topic>
-    <!-- Frames -->
-    <frame_id>base_footprint</frame_id>
-    <!-- IMPORTANT FIX -->
-    <command_timeout>0.5</command_timeout>
-    <publish_tf>true</publish_tf>
-  </plugin>
-</gazebo>
--->
-  <!-- Gazebo materials -->
+  <!-- ================= GAZEBO MATERIALS & PHYSICS ================= -->
   <gazebo reference="base_link">
     <material>Gazebo/Blue</material>
   </gazebo>
-  <gazebo reference="right_wheel_link">
-    <material>Gazebo/Grey</material>
-  </gazebo>
-  <gazebo reference="left_wheel_link">
-    <material>Gazebo/Grey</material>
-  </gazebo>
-  <gazebo reference="castor_wheel_link1">
-    <material>Gazebo/Grey</material>
-  </gazebo>
-<gazebo>
-  <plugin
-    filename="gz-sim-joint-state-publisher-system"
-    name="gz::sim::systems::JointStatePublisher">
-    <joint_name>base_to_left_wheel</joint_name>
-    <joint_name>base_to_right_wheel</joint_name>
-  </plugin>
+<gazebo reference="left_wheel_link">
+  <mu1>50.0</mu1>
+  <mu2>50.0</mu2>
+  <kp>1000000.0</kp>
+  <kd>100.0</kd>
 </gazebo>
+<gazebo reference="right_wheel_link">
+  <mu1>50.0</mu1>
+  <mu2>50.0</mu2>
+  <kp>1000000.0</kp>
+  <kd>100.0</kd>
+</gazebo>
+<gazebo reference="castor_wheel_link">
+  <mu1>0.0</mu1>
+  <mu2>0.0</mu2>
+  <slip1>1.0</slip1>
+  <slip2>1.0</slip2>
+</gazebo>
+  <!--
+    The native Gazebo diff-drive plugin has been removed from here.
+    The 'diff_drive_controller' in ros2_control handles the robot movements.
+    The gz_ros2_control plugin itself is declared in mobile_base.ros2_control.xacro.
+  -->
 </robot>

File: src/my_robot_description/urdf/my_robot.urdf.xacro (robot description, xacro)
@@ -1,11 +1,15 @@
 <?xml version='1.0'?>
-<!-- Dummy commit -->
-<robot name='my_robot' xmlns:xacro='http://www.ros.org/wiki/xacro'>
-<xacro:include filename='common_properties.xacro'/>
-<xacro:include filename='mobile_base.xacro'/>
-<xacro:include filename='mobile_base.ros2_control.xacro'/>
-<xacro:include filename='camera.xacro'/>
-<xacro:include filename='lidar.xacro'/>
-<xacro:include filename='imu.xacro'/>
-<!-- <xacro:include filename='mobile_base_gazebo.xacro'/> -->
+<robot name='my_robot' xmlns:xacro='http://ros.org'>
+  <xacro:arg name='use_ros2_control' default='false'/>
+  <xacro:include filename='common_properties.xacro'/>
+  <xacro:include filename='mobile_base.xacro'/>
+  <!-- Materials/friction apply regardless of control mode -->
+  <xacro:include filename='mobile_base_gazebo.xacro'/>
+  <!-- FIX: Added $(arg ...) inside the curly braces to evaluate the argument -->
+  <xacro:if value='$(arg use_ros2_control)'>
+    <xacro:include filename='mobile_base.ros2_control.xacro'/>
+  </xacro:if>
+  <xacro:include filename='camera.xacro'/>
+  <xacro:include filename='lidar.xacro'/>
+  <xacro:include filename='imu.xacro'/>
 </robot>
